File: _autosave-usb-toolbag.kicad_pcb (KiCad board)
At the start: 4 copper layers, 49.8 x 17.9 mm, 33 parts, among them J1 USB_A, J2 Conn_01x25_Pin, SW1 KMR2, SW2 KMR2, U1 29F32G08-TSOP48, U2 RT9080-3.3, U3 RP2040, U4 8MB QSPI, Y1 12MHz

Commit message: I seriously can't help myself...an artist is never done tweaking things...
Parts:
- moved C4 2.00 mm to (115.4, 106.3), turned to 0 degrees
- moved R6 0.93 mm to (120.8, 109.1)
- moved C5 0.73 mm to (115.8, 110.4), turned to 90 degrees
- moved R2 0.72 mm to (131.0, 115.5)
- moved R1 0.42 mm to (128.3, 115.9)
- moved C6 0.33 mm to (126.1, 115.9)
Routing:
- net /GPIO16: track 19.9 -> 21.0 mm
- net Net-(U3-XOUT): track 9.29 -> 8.39 mm
- net /GPIO17: track 21.3 -> 22.2 mm
- net Net-(U3-USB_DM): track 4.81 -> 4.06 mm
- net Net-(J1-D-): track 9.53 -> 10.2 mm
